File: gsd/love.kicad_pcb (KiCad board)
At the start: 2 copper layers, 285.8 x 94.9 mm, 75 parts, among them U2 Raspberry_Pi_Pico

Commit message: renaming the project folder name
Parts:
- removed the G*** at (284.8, 253.8)
- removed the G*** at (231.5, 253.8)
- added G***: LOGO, graphics:gsd, F.Cu at (263.3, 254.3)
Other:
- outline, holes or cut-outs redrawn
- board text removed: "Patrick & Natalie 02/18/2022"
