File: love/love.kicad_pcb (KiCad board)
At the start: 2 copper layers, 285.8 x 94.9 mm, 75 parts, among them U2 Raspberry_Pi_Pico

Commit message: v2
Routing:
- removed copper zone on B.Cu, net (none)
- removed copper zone on F.Cu, net (none)
Changed lines of the file:
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@@
     (effects (font (size 3 3) (thickness 0.2) bold) (justify bottom))
+  )
+  (dimension (type aligned) (layer "F.Cu")
+    (pts (xy 135 300) (xy 114.2 300))
+    (height 6.5)
+    (gr_text "20.8000 mm" (at 124.6 290.2) (layer "F.Cu")
+      (effects (font (size 3 3) (thickness 0.3)))
+    )
+    (format (prefix "") (suffix "") (units 3) (units_format 1) (precision 4))
+    (style (thickness 0.2) (arrow_length 1.27) (text_position_mode 0) (extension_height 0.58642) (extension_offset 0.5) keep_text_aligned)
+  )
+  (dimension (type aligned) (layer "F.Cu")
+    (pts (xy 135 300) (xy 135 314))
+    (height -6.8)
+    (gr_text "14.0000 mm" (at 140 307 90) (layer "F.Cu")
+      (effects (font (size 1.5 1.5) (thickness 0.3)))
+    )
+    (format (prefix "") (suffix "") (units 3) (units_format 1) (precision 4))
+    (style (thickness 0.2) (arrow_length 1.27) (text_position_mode 0) (extension_height 0.58642) (extension_offset 0.5) keep_text_aligned)
+  )
+  (dimension (type aligned) (layer "F.Cu")
+    (pts (xy 117.2 219.1) (xy 117.2 314))
+    (height 18.14)
+    (gr_text "94.9000 mm" (at 95.76 266.55 90) (layer "F.Cu")
+      (effects (font (size 3 3) (thickness 0.3)))
+    )
+    (format (prefix "") (suffix "") (units 3) (units_format 1) (precision 4))
+    (style (thickness 0.2) (arrow_length 1.27) (text_position_mode 0) (extension_height 0.58642) (extension_offset 0.5) keep_text_aligned)
+  )
+  (dimension (type aligned) (layer "F.Cu")
+    (pts (xy 156.8 219.1) (xy 114.3 219.1))
+    (height 1.9)
+    (gr_text "42.5000 mm" (at 135.55 215.4) (layer "F.Cu")
+      (effects (font (size 1.5 1.5) (thickness 0.3)))
+    )
+    (format (prefix "") (suffix "") (units 3) (units_format 1) (precision 4))
+    (style (thickness 0.2) (arrow_length 1.27) (text_position_mode 0) (extension_height 0.58642) (extension_offset 0.5) keep_text_aligned)
+  )
+  (dimension (type aligned) (layer "F.Cu")
+    (pts (xy 109.0398 250.350008) (xy 108.9948 221.800008))
+    (height 0.0052)
+    (gr_text "28.5500 mm" (at 110.822498 236.072163 -89.90969149) (layer "F.Cu")
+      (effects (font (size 1.5 1.5) (thickness 0.3)))
+    )
+    (format (prefix "") (suffix "") (units 3) (units_format 1) (precision 4))
+    (style (thickness 0.2) (arrow_length 1.27) (text_position_mode 0) (extension_height 0.58642) (extension_offset 0.5) keep_text_aligned)
+  )
+  (dimension (type aligned) (layer "F.Cu")
+    (pts (xy 114.3 222) (xy 400.05 221.95))
+    (height -13.516215)
+    (gr_text "285.7500 mm" (at 257.172058 205.158785 0.01002550812) (layer "F.Cu")
+      (effects (font (size 3 3) (thickness 0.3)))
+    )
+    (format (prefix "") (suffix "") (units 3) (units_format 1) (precision 4))
+    (style (thickness 0.2) (arrow_length 1.27) (text_position_mode 0) (extension_height 0.58642) (extension_offset 0.5) keep_text_aligned)
+  )
+  (dimension (type aligned) (layer "Edge.Cuts")
+    (pts (xy 357.505 247.65) (xy 400.1 247.7))
+    (height -22.573028)
+    (gr_text "42.5950 mm" (at 378.830347 223.951989 359.9327436) (layer "Edge.Cuts")
+      (effects (font (size 1 1) (thickness 0.15)))
+    )
+    (format (prefix "") (suffix "") (units 3) (units_format 1) (precision 4))
+    (style (thickness 0.1) (arrow_length 1.27) (text_position_mode 0) (extension_height 0.58642) (extension_offset 0.5) keep_text_aligned)
+  )
+  (dimension (type aligned) (layer "Edge.Cuts")
+    (pts (xy 357.5 247.75) (xy 357.5 228.6))
+    (height 52)
+    (gr_text "19.1500 mm" (at 408.35 238.175 90) (layer "Edge.Cuts")
+      (effects (font (size 1 1) (thickness 0.15)))
+    )
+    (format (prefix "") (suffix "") (units 3) (units_format 1) (precision 4))
+    (style (thickness 0.1) (arrow_length 1.27) (text_position_mode 0) (extension_height 0.58642) (extension_offset 0.5) keep_text_aligned)
+  )
+  (dimension (type aligned) (layer "Edge.Cuts")
+    (pts (xy 377.3 300.1) (xy 400.1 300.1))
+    (height -7.4)
+    (gr_text "22.8000 mm" (at 388.7 291.55) (layer "Edge.Cuts")
+      (effects (font (size 1 1) (thickness 0.15)))
+    )
+    (format (prefix "") (suffix "") (units 3) (units_format 1) (precision 4))
+    (style (thickness 0.1) (arrow_length 1.27) (text_position_mode 0) (extension_height 0.58642) (extension_offset 0.5) keep_text_aligned)
+  )
+  (dimension (type aligned) (layer "Edge.Cuts")
+    (pts (xy 377.3 300.1) (xy 377.3 314))
+    (height -32.6)
+    (gr_text "13.9000 mm" (at 408.75 307.05 90) (layer "Edge.Cuts")
+      (effects (font (size 1 1) (thickness 0.15)))
+    )
+    (format (prefix "") (suffix "") (units 3) (units_format 1) (precision 4))
+    (style (thickness 0.1) (arrow_length 1.27) (text_position_mode 0) (extension_height 0.58642) (extension_offset 0.5) keep_text_aligned)
   )
   (segment (start 233.3625 252.4125) (end 238.125 257.175) (width 0.25) (layer "F.Cu") (net 1))
@@
   (segment (start 300.355 293.5625) (end 299.6925 292.9) (width 0.25) (layer "B.Cu") (net 54))
   (segment (start 276.225 283.845) (end 266.065 273.685) (width 0.25) (layer "B.Cu") (net 54))
-  (zone (net 0) (net_name "") (layers "F&B.Cu") (hatch edge 0.5)
-    (connect_pads (clearance 0.5))
-    (min_thickness 0.25) (filled_areas_thickness no)
-    (fill yes (thermal_gap 0.5) (thermal_bridge_width 0.5) (island_removal_mode 1) (island_area_min 10))
-    (polygon
-      (pts
-        (xy 107 189.4)
-        (xy 104.05 352.9)
-        (xy 431.6 351.15)
-        (xy 427.5 186.2)
-      )
-    )
-  )
 )
