File: yuri_v2/yuri_v2.kicad_pcb (KiCad board)
At the start: 2 copper layers, 303.4 x 95.4 mm, 79 parts, among them SW1 RotaryEncoder_Switch, SW2 RotaryEncoder_Switch, SW4 SW_PUSH, U1 Elite-C

Commit message: added a submitted order
Parts:
- added G***: LOGO, graphics:growling-gsd, B.Cu at (204.8, 111.0)
- moved G*** 5.32 mm to (203.1, 116.1)
Routing:
- added copper zone on B.Cu, net Reset
- added copper zone on F.Cu, net Reset
- removed copper zone on B.Cu, net (none)
- removed copper zone on F.Cu, net (none)
Other:
- board size 303.4 x 95.4 mm -> 303.4 x 93 mm

Commit message: adding the traditional 84 key but for somereason i named it 104
Routing:
- removed copper zone on B.Cu, net Reset
- removed copper zone on F.Cu, net Reset
